File: Meshtastic-basestation-repeater.kicad_sch (KiCad schematic)
At the start: 7 parts

Commit message: Protection diode
Parts:
- added D1: SR540, symbol pspice:DIODE
- J1: renamed from J?; value Screw_Terminal_01x02 -> DC IN
- J2: renamed from J?; value Conn_01x03 -> GPS voltage
- J3: renamed from J?; value Conn_01x04 -> GPS
- gave numbers to parts that had none: 4
Connections:
- net GND: now also J3.4 (Pin_4)
- net VDC: now also D1.2 (A); no longer J1.1 (Pin_1)
- new net: D1.1 (K), J1.1 (Pin_1)
